File: hex-debouncer/hex-debouncer.kicad_pcb (KiCad board)
At the start: 2 copper layers, 37 parts, among them J1 Conn_01x08, SW1 A, SW2 B, SW3 C, SW4 D, SW5 E, SW6 F, U1 74HC14

Commit message: up
Parts:
- added J2: Conn_01x08, Connector_PinHeader_2.54mm:PinHeader_1x08_P2.54mm_Vertical, F.Cu at (119.4, 100.3)
Changed lines of the file:
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@@
       (net 2 "GND") (pinfunction "1") (pintype "input"))
+  )
+  (footprint "Connector_PinHeader_2.54mm:PinHeader_1x08_P2.54mm_Vertical" (layer "F.Cu")
+    (at 119.38 100.33 -90)
+    (descr "Through hole straight pin header, 1x08, 2.54mm pitch, single row")
+    (tags "Through hole pin header THT 1x08 2.54mm single row")
+    (property "Sheetfile" "hex-debouncer.kicad_sch")
+    (property "Sheetname" "")
+    (attr through_hole)
+    (fp_text reference "J2" (at 0 -2.33 90) (layer "F.SilkS")
+      (effects (font (size 1 1) (thickness 0.15)))
+    )
+    (fp_text value "Conn_01x08" (at 0 20.11 90) (layer "F.Fab")
+      (effects (font (size 1 1) (thickness 0.15)))
+    )
+    (fp_text user "${REFERENCE}" (at 0 8.89) (layer "F.Fab")
+      (effects (font (size 1 1) (thickness 0.15)))
+    )
+    (fp_line (start -1.33 1.27) (end 1.33 1.27) (layer "F.SilkS") (width 0.12))
+    (fp_line (start -1.33 0) (end -1.33 -1.33) (layer "F.SilkS") (width 0.12))
+    (fp_line (start 1.33 1.27) (end 1.33 19.11) (layer "F.SilkS") (width 0.12))
+    (fp_line (start -1.33 1.27) (end -1.33 19.11) (layer "F.SilkS") (width 0.12))
+    (fp_line (start -1.33 19.11) (end 1.33 19.11) (layer "F.SilkS") (width 0.12))
+    (fp_line (start -1.33 -1.33) (end 0 -1.33) (layer "F.SilkS") (width 0.12))
+    (fp_line (start 1.8 19.55) (end 1.8 -1.8) (layer "F.CrtYd") (width 0.05))
+    (fp_line (start 1.8 -1.8) (end -1.8 -1.8) (layer "F.CrtYd") (width 0.05))
+    (fp_line (start -1.8 19.55) (end 1.8 19.55) (layer "F.CrtYd") (width 0.05))
+    (fp_line (start -1.8 -1.8) (end -1.8 19.55) (layer "F.CrtYd") (width 0.05))
+    (fp_line (start 1.27 -1.27) (end 1.27 19.05) (layer "F.Fab") (width 0.1))
+    (fp_line (start 1.27 19.05) (end -1.27 19.05) (layer "F.Fab") (width 0.1))
+    (fp_line (start -1.27 -0.635) (end -0.635 -1.27) (layer "F.Fab") (width 0.1))
+    (fp_line (start -1.27 19.05) (end -1.27 -0.635) (layer "F.Fab") (width 0.1))
+    (fp_line (start -0.635 -1.27) (end 1.27 -1.27) (layer "F.Fab") (width 0.1))
+    (pad "1" thru_hole rect (at 0 0 270) (size 1.7 1.7) (drill 1) (layers *.Cu *.Mask)
+      (net 8 "VCC") (pinfunction "Pin_1") (pintype "passive"))
+    (pad "2" thru_hole oval (at 0 2.54 270) (size 1.7 1.7) (drill 1) (layers *.Cu *.Mask)
+      (net 2 "GND") (pinfunction "Pin_2") (pintype "passive"))
+    (pad "3" thru_hole oval (at 0 5.08 270) (size 1.7 1.7) (drill 1) (layers *.Cu *.Mask)
+      (net 15 "A") (pinfunction "Pin_3") (pintype "passive"))
+    (pad "4" thru_hole oval (at 0 7.62 270) (size 1.7 1.7) (drill 1) (layers *.Cu *.Mask)
+      (net 16 "B") (pinfunction "Pin_4") (pintype "passive"))
+    (pad "5" thru_hole oval (at 0 10.16 270) (size 1.7 1.7) (drill 1) (layers *.Cu *.Mask)
+      (net 17 "C") (pinfunction "Pin_5") (pintype "passive"))
+    (pad "6" thru_hole oval (at 0 12.7 270) (size 1.7 1.7) (drill 1) (layers *.Cu *.Mask)
+      (net 18 "D") (pinfunction "Pin_6") (pintype "passive"))
+    (pad "7" thru_hole oval (at 0 15.24 270) (size 1.7 1.7) (drill 1) (layers *.Cu *.Mask)
+      (net 19 "E") (pinfunction "Pin_7") (pintype "passive"))
+    (pad "8" thru_hole oval (at 0 17.78 270) (size 1.7 1.7) (drill 1) (layers *.Cu *.Mask)
+      (net 20 "F") (pinfunction "Pin_8") (pintype "passive"))
+    (model "${KICAD6_3DMODEL_DIR}/Connector_PinHeader_2.54mm.3dshapes/PinHeader_1x08_P2.54mm_Vertical.wrl"
+      (offset (xyz 0 0 0))
+      (scale (xyz 1 1 1))
+      (rotate (xyz 0 0 0))
+    )
   )
   (footprint "Button_Switch_SMD:SW_SPST_PTS645" (layer "F.Cu")
@@
     )
   )
-  (gr_line (start 139.7 96.52) (end 139.7 71.12) (layer "Dwgs.User") (width 0.15))
-  (gr_line (start 78.74 71.12) (end 78.74 96.52) (layer "Dwgs.User") (width 0.15))
-  (gr_line (start 139.7 71.12) (end 78.74 71.12) (layer "Dwgs.User") (width 0.15))
-  (gr_line (start 78.74 96.52) (end 139.7 96.52) (layer "Dwgs.User") (width 0.15))
 )
