File: project_files/hex-debouncer.kicad_sch (KiCad schematic)
At the start: 38 parts, among them J1 Conn_01x08, J2 Conn_01x08, SW1 A, SW2 B, SW3 C, SW4 D, SW5 E, SW6 F, U1 74HC14

Commit message: FInalized layout
Parts:
- removed J2: Conn_01x08, Connector_PinHeader_2.54mm:PinHeader_1x08_P2.54mm_Vertical, symbol Connector_Generic:Conn_01x08
- added SW10: B, Button_Switch_THT:SW_PUSH_6mm_H8mm, symbol Switch:SW_Push
- added SW11: D, Button_Switch_THT:SW_PUSH_6mm_H8mm, symbol Switch:SW_Push
- added SW12: F, Button_Switch_THT:SW_PUSH_6mm_H8mm, symbol Switch:SW_Push
- added SW7: A, Button_Switch_THT:SW_PUSH_6mm_H8mm, symbol Switch:SW_Push
- added SW8: C, Button_Switch_THT:SW_PUSH_6mm_H8mm, symbol Switch:SW_Push
- added SW9: E, Button_Switch_THT:SW_PUSH_6mm_H8mm, symbol Switch:SW_Push
- added U2: 74HC14, Package_DIP:DIP-14_W7.62mm, symbol 74xx:74HC14
- J1: value Conn_01x08 -> UPPER
- SW1, SW2, SW3, SW4, SW5, SW6: now not fitted
Connections:
- net A: now also U2.2
- net B: now also U2.4
- net C: now also U2.6
- net D: now also U1.12, U2.12; no longer U1.8
- net E: now also U2.10
- net F: now also U1.8, U2.8; no longer U1.12
- net GND: now also SW10.1, SW11.1, SW12.1, SW7.1, SW8.1, SW9.1, U2.7 (GND)
- net VCC: now also U2.14 (VCC)
- net BUT_C: now reaches C3.1, D3.1 (K), R7.1, U1.5
- net BUT_C: now also U2.5
- net at D3.2 (A), R5.2, R7.2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: now also SW8.2
- net BUT_D: now reaches C6.1, D6.1 (K), R12.1, U1.13
- net BUT_D: now also U2.13
- net at D4.2 (A), R6.2, R8.2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: now also SW11.2
- net BUT_A: now reaches C1.1, D1.1 (K), R3.1, U1.1
- net BUT_A: now also U2.1
- net BUT_B: now reaches C2.1, D2.1 (K), R4.1, U1.3
- net BUT_B: now also U2.3
- net at D2.2 (A), R2.2, R4.2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: now also SW10.2
- net at D6.2 (A), R10.2, R12.2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: now also SW12.2
- net at D5.2 (A), R11.2, R9.2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: now also SW9.2
- net BUT_F: now reaches C4.1, D4.1 (K), R8.1, U1.9
- net BUT_F: now also U2.9
- net at D1.2 (A), R1.2, R3.2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: now also SW7.2
- net BUT_E: now reaches C5.1, D5.1 (K), R11.1, U1.11
- net BUT_E: now also U2.11
Other:
- title: (none) -> Push-Buttons module with debouncing
- moved on the sheet: C1, C2, C3, C4, C5, C6, C7, D1, D2, D3, D4, D5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
